Commit message: Add simulator sensor bringup and RViz fixes

File: cyberdog_robot/cyberdog_description/xacro/gazebo.xacro (robot description, xacro)
@@ -30,39 +30,200 @@
         </sensor>
     </gazebo>
+    <gazebo reference="RGB_camera_link">
+        <sensor name="rgb_camera" type="camera">
+            <always_on>true</always_on>
+            <update_rate>30.0</update_rate>
+            <visualize>true</visualize>
+            <pose>0 0 0 0 0 0</pose>
+            <camera name="rgb_camera_sensor">
+                <horizontal_fov>1.3962634</horizontal_fov>
+                <image>
+                    <width>640</width>
+                    <height>480</height>
+                    <format>R8G8B8</format>
+                </image>
+                <clip>
+                    <near>0.02</near>
+                    <far>300</far>
+                </clip>
+                <noise>
+                    <type>gaussian</type>
+                    <mean>0.0</mean>
+                    <stddev>0.007</stddev>
+                </noise>
+            </camera>
+            <plugin name="rgb_camera_controller" filename="libgazebo_ros_camera.so">
+                <ros>
+                    <namespace>/rgb_camera</namespace>
+                    <remapping>rgb_camera/image_raw:=image_raw</remapping>
+                    <remapping>rgb_camera/camera_info:=camera_info</remapping>
+                </ros>
+                <camera_name>rgb_camera</camera_name>
+                <frame_name>RGB_camera_link</frame_name>
+            </plugin>
+        </sensor>
+    </gazebo>
+    <gazebo reference="D435_camera_link">
+        <sensor name="depth_camera" type="depth">
+            <always_on>true</always_on>
+            <update_rate>30.0</update_rate>
+            <visualize>true</visualize>
+            <pose>0 0 0 0 0 0</pose>
+            <camera name="depth_camera_sensor">
+                <horizontal_fov>1.3962634</horizontal_fov>
+                <image>
+                    <width>640</width>
+                    <height>480</height>
+                    <format>R8G8B8</format>
+                </image>
+                <depth_camera/>
+                <clip>
+                    <near>0.02</near>
+                    <far>10.0</far>
+                </clip>
+                <noise>
+                    <type>gaussian</type>
+                    <mean>0.0</mean>
+                    <stddev>0.007</stddev>
+                </noise>
+            </camera>
+            <plugin name="depth_camera_controller" filename="libgazebo_ros_camera.so">
+                <ros>
+                    <namespace>/d435_camera</namespace>
+                    <remapping>d435_depth/image_raw:=depth/image_raw</remapping>
+                    <remapping>d435_depth/depth/image_raw:=depth/depth_image_raw</remapping>
+                    <remapping>d435_depth/camera_info:=depth/camera_info</remapping>
+                    <remapping>d435_depth/depth/camera_info:=depth/depth_camera_info</remapping>
+                    <remapping>d435_depth/points:=depth/points</remapping>
+                </ros>
+                <camera_name>d435_depth</camera_name>
+                <frame_name>D435_camera_link</frame_name>
+                <min_depth>0.1</min_depth>
+                <max_depth>10.0</max_depth>
+            </plugin>
+        </sensor>
+    </gazebo>
+    <gazebo reference="AI_camera_link">
+        <sensor name="stereo_camera" type="multicamera">
+            <always_on>true</always_on>
+            <update_rate>30.0</update_rate>
+            <visualize>true</visualize>
+            <camera name="left">
+                <horizontal_fov>1.3962634</horizontal_fov>
+                <image>
+                    <width>640</width>
+                    <height>480</height>
+                    <format>R8G8B8</format>
+                </image>
+                <clip>
+                    <near>0.02</near>
+                    <far>300</far>
+                </clip>
+                <noise>
+                    <type>gaussian</type>
+                    <mean>0.0</mean>
+                    <stddev>0.007</stddev>
+                </noise>
+            </camera>
+            <camera name="right">
+                <pose>0 -0.05 0 0 0 0</pose>
+                <horizontal_fov>1.3962634</horizontal_fov>
+                <image>
+                    <width>640</width>
+                    <height>480</height>
+                    <format>R8G8B8</format>
+                </image>
+                <clip>
+                    <near>0.02</near>
+                    <far>300</far>
+                </clip>
+                <noise>
+                    <type>gaussian</type>
+                    <mean>0.0</mean>
+                    <stddev>0.007</stddev>
+                </noise>
+            </camera>
+            <plugin name="stereo_camera_controller" filename="libgazebo_ros_camera.so">
+                <ros>
+                    <namespace>/ai_camera</namespace>
+                    <remapping>stereo/left/image_raw:=left/image_raw</remapping>
+                    <remapping>stereo/right/image_raw:=right/image_raw</remapping>
+                    <remapping>stereo/left/camera_info:=left/camera_info</remapping>
+                    <remapping>stereo/right/camera_info:=right/camera_info</remapping>
+                </ros>
+                <camera_name>stereo</camera_name>
+                <frame_name>AI_camera_link</frame_name>
+            </plugin>
+        </sensor>
+    </gazebo>
     <xacro:if value="$(arg USE_LIDAR)">
         <gazebo reference="lidar_link">
-        <sensor name="realsense" type="ray">
-            <always_on>true</always_on>
-            <visualize>true</visualize>
-            <pose>0.0 0 0.0 0 0 0</pose>
-            <update_rate>5</update_rate>
-            <ray>
-            <scan>
-                <horizontal>
-                <samples>180</samples>
-                <resolution>1.000000</resolution>
-                <min_angle>-1.5700</min_angle>
-                <max_angle>1.5700</max_angle>
-                </horizontal>
-            </scan>
-            <range>
-                <min>0.01</min>
-                <max>12.00</max>
-                <resolution>0.015000</resolution>
-            </range>
-            <noise>
-                <type>gaussian</type>
-                <mean>0.0</mean>
-                <stddev>0.01</stddev>
-            </noise>
-            </ray>
-            <plugin name="cyberdog_laserscan" filename="libgazebo_ros_ray_sensor.so">
-            <ros>
-                <remapping>~/out:=scan</remapping>
-            </ros>
-            <output_type>sensor_msgs/LaserScan</output_type>
-            <frame_name>lidar_link</frame_name>
-            </plugin>
-        </sensor>
+            <sensor name="lidar_ray" type="ray">
+                <always_on>true</always_on>
+                <visualize>true</visualize>
+                <pose>0 0 0 0 0 0</pose>
+                <update_rate>5</update_rate>
+                <ray>
+                    <scan>
+                        <horizontal>
+                            <samples>180</samples>
+                            <resolution>1.0</resolution>
+                            <min_angle>-1.5700</min_angle>
+                            <max_angle>1.5700</max_angle>
+                        </horizontal>
+                    </scan>
+                    <range>
+                        <min>0.01</min>
+                        <max>12.0</max>
+                        <resolution>0.015</resolution>
+                    </range>
+                    <noise>
+                        <type>gaussian</type>
+                        <mean>0.0</mean>
+                        <stddev>0.01</stddev>
+                    </noise>
+                </ray>
+                <plugin name="cyberdog_laserscan" filename="libgazebo_ros_ray_sensor.so">
+                    <ros>
+                        <namespace>/lidar</namespace>
+                        <remapping>~/out:=scan</remapping>
+                    </ros>
+                    <output_type>sensor_msgs/LaserScan</output_type>
+                    <frame_name>lidar_link</frame_name>
+                </plugin>
+            </sensor>
+            <sensor name="lidar_gpu_ray" type="gpu_ray">
+                <always_on>true</always_on>
+                <visualize>true</visualize>
+                <pose>0 0 0 0 0 0</pose>
+                <update_rate>5</update_rate>
+                <ray>
+                    <scan>
+                        <horizontal>
+                            <samples>180</samples>
+                            <resolution>1.0</resolution>
+                            <min_angle>-1.5700</min_angle>
+                            <max_angle>1.5700</max_angle>
+                        </horizontal>
+                    </scan>
+                    <range>
+                        <min>0.01</min>
+                        <max>12.0</max>
+                    </range>
+                    <noise>
+                        <type>gaussian</type>
+                        <mean>0.0</mean>
+                        <stddev>0.01</stddev>
+                    </noise>
+                </ray>
+                <plugin name="cyberdog_gpu_laserscan" filename="libgazebo_ros_ray_sensor.so">
+                    <ros>
+                        <namespace>/lidar_gpu</namespace>
+                        <remapping>~/out:=scan</remapping>
+                    </ros>
+                    <output_type>sensor_msgs/LaserScan</output_type>
+                    <frame_name>lidar_link</frame_name>
+                </plugin>
+            </sensor>
         </gazebo>
     </xacro:if>
@@ -70,36 +231,64 @@
     <gazebo reference="FR_knee">
         <sensor name="FR_foot_contact" type="contact">
-        <update_rate>100</update_rate>
-        <plugin name="contactPlugin" filename="libfoot_contact_plugin.so"/>
-        <contact>
-            <collision>FR_knee_fixed_joint_lump__FR_foot_collision_2</collision>
-        </contact>
+            <update_rate>100</update_rate>
+            <plugin name="contactPlugin" filename="libfoot_contact_plugin.so"/>
+            <plugin name="FR_bumper_controller" filename="libgazebo_ros_bumper.so">
+                <ros>
+                    <namespace>/foot_contact</namespace>
+                    <remapping>bumper_states:=fr</remapping>
+                </ros>
+                <frame_name>FR_knee</frame_name>
+            </plugin>
+            <contact>
+                <collision>FR_knee_fixed_joint_lump__FR_foot_collision_2</collision>
+            </contact>
         </sensor>
     </gazebo>
     <gazebo reference="FL_knee">
         <sensor name="FL_foot_contact" type="contact">
-        <update_rate>100</update_rate>
-        <plugin name="contactPlugin" filename="libfoot_contact_plugin.so"/>
-        <contact>
-            <collision>FL_knee_fixed_joint_lump__FL_foot_collision_2</collision>
-        </contact>
+            <update_rate>100</update_rate>
+            <plugin name="contactPlugin" filename="libfoot_contact_plugin.so"/>
+            <plugin name="FL_bumper_controller" filename="libgazebo_ros_bumper.so">
+                <ros>
+                    <namespace>/foot_contact</namespace>
+                    <remapping>bumper_states:=fl</remapping>
+                </ros>
+                <frame_name>FL_knee</frame_name>
+            </plugin>
+            <contact>
+                <collision>FL_knee_fixed_joint_lump__FL_foot_collision_2</collision>
+            </contact>
         </sensor>
     </gazebo>
     <gazebo reference="RR_knee">
         <sensor name="RR_foot_contact" type="contact">
-        <update_rate>100</update_rate>
-        <plugin name="contactPlugin" filename="libfoot_contact_plugin.so"/>
-        <contact>
-            <collision>RR_knee_fixed_joint_lump__RR_foot_collision_2</collision>
-        </contact>
+            <update_rate>100</update_rate>
+            <plugin name="contactPlugin" filename="libfoot_contact_plugin.so"/>
+            <plugin name="RR_bumper_controller" filename="libgazebo_ros_bumper.so">
+                <ros>
+                    <namespace>/foot_contact</namespace>
+                    <remapping>bumper_states:=rr</remapping>
+                </ros>
+                <frame_name>RR_knee</frame_name>
+            </plugin>
+            <contact>
+                <collision>RR_knee_fixed_joint_lump__RR_foot_collision_2</collision>
+            </contact>
         </sensor>
     </gazebo>
     <gazebo reference="RL_knee">
         <sensor name="RL_foot_contact" type="contact">
-        <update_rate>100</update_rate>
-        <plugin name="contactPlugin" filename="libfoot_contact_plugin.so"/>
-        <contact>
-            <collision>RL_knee_fixed_joint_lump__RL_foot_collision_2</collision>
-        </contact>
+            <update_rate>100</update_rate>
+            <plugin name="contactPlugin" filename="libfoot_contact_plugin.so"/>
+            <plugin name="RL_bumper_controller" filename="libgazebo_ros_bumper.so">
+                <ros>
+                    <namespace>/foot_contact</namespace>
+                    <remapping>bumper_states:=rl</remapping>
+                </ros>
+                <frame_name>RL_knee</frame_name>
+            </plugin>
+            <contact>
+                <collision>RL_knee_fixed_joint_lump__RL_foot_collision_2</collision>
+            </contact>
         </sensor>
     </gazebo>

File: cyberdog_robot/cyberdog_description/xacro/leg.xacro (robot description, xacro)
@@ -209,5 +209,5 @@
                 <material name="orange" />
             </visual>
-            <collision>
+            <collision name="${name}_foot_collision">
                 <origin rpy="0 0 0" xyz="0 0 0" />
                 <geometry>
