Commit message: [Feat]: add optional simulator camera bringup and launch arg forwarding
Functions updated:

- forward simulator launch args from launchsim to gazebo and visual scripts

- add optional RealSense, stereo, and AI camera launch arguments across gazebo, description, and visual pipelines

- add camera frames and conditional gazebo sensor definitions in cyberdog_description xacro files

- add simulator build/package dependency updates for xacro and gazebo plugins

- add lcm cmake fallback lookup under /usr/local for source installs

File: cyberdog_robot/cyberdog_description/xacro/gazebo.xacro (robot description, xacro)
@@ -228,4 +228,229 @@
         </gazebo>
     </xacro:if>
+    <xacro:if value="$(arg USE_REALSENSE_CAMERA)">
+        <gazebo reference="camera_infra1_frame">
+            <sensor name="infra1_camera" type="camera">
+                <always_on>true</always_on>
+                <update_rate>30</update_rate>
+                <visualize>false</visualize>
+                <camera>
+                    <horizontal_fov>1.518</horizontal_fov>
+                    <image>
+                        <width>848</width>
+                        <height>480</height>
+                        <format>L8</format>
+                    </image>
+                    <clip>
+                        <near>0.20</near>
+                        <far>10.0</far>
+                    </clip>
+                </camera>
+                <plugin filename="libgazebo_ros_camera.so" name="infra1_camera_plugin">
+                    <ros>
+                        <remapping>infra1/image_raw:=/camera/infra1/image_rect_raw</remapping>
+                        <remapping>infra1/camera_info:=/camera/infra1/camera_info</remapping>
+                    </ros>
+                    <camera_name>infra1</camera_name>
+                    <frame_name>camera_infra1_optical_frame</frame_name>
+                </plugin>
+            </sensor>
+        </gazebo>
+        <gazebo reference="camera_infra2_frame">
+            <sensor name="infra2_camera" type="camera">
+                <always_on>true</always_on>
+                <update_rate>30</update_rate>
+                <visualize>false</visualize>
+                <camera>
+                    <horizontal_fov>1.518</horizontal_fov>
+                    <image>
+                        <width>848</width>
+                        <height>480</height>
+                        <format>L8</format>
+                    </image>
+                    <clip>
+                        <near>0.20</near>
+                        <far>10.0</far>
+                    </clip>
+                </camera>
+                <plugin filename="libgazebo_ros_camera.so" name="infra2_camera_plugin">
+                    <ros>
+                        <remapping>infra2/image_raw:=/camera/infra2/image_rect_raw</remapping>
+                        <remapping>infra2/camera_info:=/camera/infra2/camera_info</remapping>
+                    </ros>
+                    <camera_name>infra2</camera_name>
+                    <frame_name>camera_infra2_optical_frame</frame_name>
+                </plugin>
+            </sensor>
+        </gazebo>
+        <gazebo reference="camera_depth_frame">
+            <sensor name="depth_camera" type="depth">
+                <always_on>true</always_on>
+                <update_rate>30</update_rate>
+                <visualize>false</visualize>
+                <camera>
+                    <horizontal_fov>1.518</horizontal_fov>
+                    <image>
+                        <width>848</width>
+                        <height>480</height>
+                        <format>R8G8B8</format>
+                    </image>
+                    <depth_camera>
+                    </depth_camera>
+                    <clip>
+                        <near>0.20</near>
+                        <far>10.0</far>
+                    </clip>
+                </camera>
+                <plugin filename="libgazebo_ros_camera.so" name="depth_camera_plugin">
+                    <ros>
+                        <remapping>depth_camera/image_raw:=/camera/depth/raw/image_raw</remapping>
+                        <remapping>depth_camera/camera_info:=/camera/depth/raw/camera_info</remapping>
+                        <remapping>depth_camera/depth/image_raw:=/camera/depth/image_rect_raw</remapping>
+                        <remapping>depth_camera/depth/camera_info:=/camera/depth/camera_info</remapping>
+                        <remapping>depth_camera/points:=/camera/depth/points</remapping>
+                    </ros>
+                    <camera_name>depth_camera</camera_name>
+                    <frame_name>camera_depth_optical_frame</frame_name>
+                    <min_depth>0.20</min_depth>
+                    <max_depth>10.0</max_depth>
+                </plugin>
+            </sensor>
+        </gazebo>
+        <gazebo reference="camera_imu_frame">
+            <gravity>true</gravity>
+            <sensor name="camera_imu_sensor" type="imu">
+                <always_on>true</always_on>
+                <update_rate>500</update_rate>
+                <visualize>false</visualize>
+                <plugin filename="libgazebo_ros_imu_sensor.so" name="camera_imu_plugin">
+                    <ros>
+                        <remapping>~/out:=/camera/imu</remapping>
+                    </ros>
+                </plugin>
+            </sensor>
+        </gazebo>
+    </xacro:if>
+    <xacro:if value="$(arg USE_STEREO_CAMERA)">
+        <gazebo reference="left_fisheye_camera_link">
+            <sensor name="left_fisheye" type="wideanglecamera">
+                <always_on>true</always_on>
+                <update_rate>30</update_rate>
+                <visualize>false</visualize>
+                <camera>
+                    <horizontal_fov>2.548</horizontal_fov>
+                    <image>
+                        <width>640</width>
+                        <height>480</height>
+                        <format>R8G8B8</format>
+                    </image>
+                    <clip>
+                        <near>0.08</near>
+                        <far>15.0</far>
+                    </clip>
+                    <lens>
+                        <type>equidistant</type>
+                        <scale_to_hfov>true</scale_to_hfov>
+                        <env_texture_size>1024</env_texture_size>
+                    </lens>
+                </camera>
+                <plugin filename="libgazebo_ros_camera.so" name="left_fisheye_plugin">
+                    <ros>
+                        <remapping>left_fisheye/image_raw:=/image_left</remapping>
+                        <remapping>left_fisheye/camera_info:=/image_left/camera_info</remapping>
+                    </ros>
+                    <camera_name>left_fisheye</camera_name>
+                    <frame_name>left_fisheye_camera_optical_frame</frame_name>
+                </plugin>
+            </sensor>
+        </gazebo>
+        <gazebo reference="right_fisheye_camera_link">
+            <sensor name="right_fisheye" type="wideanglecamera">
+                <always_on>true</always_on>
+                <update_rate>30</update_rate>
+                <visualize>false</visualize>
+                <camera>
+                    <horizontal_fov>2.548</horizontal_fov>
+                    <image>
+                        <width>640</width>
+                        <height>480</height>
+                        <format>R8G8B8</format>
+                    </image>
+                    <clip>
+                        <near>0.08</near>
+                        <far>15.0</far>
+                    </clip>
+                    <lens>
+                        <type>equidistant</type>
+                        <scale_to_hfov>true</scale_to_hfov>
+                        <env_texture_size>1024</env_texture_size>
+                    </lens>
+                </camera>
+                <plugin filename="libgazebo_ros_camera.so" name="right_fisheye_plugin">
+                    <ros>
+                        <remapping>right_fisheye/image_raw:=/image_right</remapping>
+                        <remapping>right_fisheye/camera_info:=/image_right/camera_info</remapping>
+                    </ros>
+                    <camera_name>right_fisheye</camera_name>
+                    <frame_name>right_fisheye_camera_optical_frame</frame_name>
+                </plugin>
+            </sensor>
+        </gazebo>
+        <gazebo reference="RGB_camera_link">
+            <sensor name="rgb_camera" type="camera">
+                <always_on>true</always_on>
+                <update_rate>30</update_rate>
+                <visualize>false</visualize>
+                <camera>
+                    <horizontal_fov>1.22</horizontal_fov>
+                    <image>
+                        <width>1280</width>
+                        <height>720</height>
+                        <format>R8G8B8</format>
+                    </image>
+                    <clip>
+                        <near>0.03</near>
+                        <far>20.0</far>
+                    </clip>
+                </camera>
+                <plugin filename="libgazebo_ros_camera.so" name="rgb_camera_plugin">
+                    <ros>
+                        <remapping>rgb/image_raw:=/image_rgb</remapping>
+                        <remapping>rgb/camera_info:=/image_rgb/camera_info</remapping>
+                    </ros>
+                    <camera_name>rgb</camera_name>
+                    <frame_name>rgb_camera_optical_frame</frame_name>
+                </plugin>
+            </sensor>
+        </gazebo>
+    </xacro:if>
+    <xacro:if value="$(arg USE_AI_CAMERA)">
+        <gazebo reference="AI_camera_link">
+            <sensor name="ai_camera" type="camera">
+                <always_on>true</always_on>
+                <update_rate>15</update_rate>
+                <visualize>false</visualize>
+                <camera>
+                    <horizontal_fov>1.13</horizontal_fov>
+                    <image>
+                        <width>640</width>
+                        <height>480</height>
+                        <format>R8G8B8</format>
+                    </image>
+                    <clip>
+                        <near>0.05</near>
+                        <far>20.0</far>
+                    </clip>
+                </camera>
+                <plugin filename="libgazebo_ros_camera.so" name="ai_camera_plugin">
+                    <ros>
+                        <remapping>ai/image_raw:=/image</remapping>
+                        <remapping>ai/camera_info:=/image/camera_info</remapping>
+                    </ros>
+                    <camera_name>ai</camera_name>
+                    <frame_name>ai_camera_optical_frame</frame_name>
+                </plugin>
+            </sensor>
+        </gazebo>
+    </xacro:if>
     <!-- Foot contacts. -->
     <gazebo reference="FR_knee">

File: cyberdog_robot/cyberdog_description/xacro/robot.xacro (robot description, xacro)
@@ -3,4 +3,7 @@
     <xacro:arg name="ROBOT" default="cyber_dog" />
     <xacro:arg name="USE_LIDAR" default="false" />
+    <xacro:arg name="USE_REALSENSE_CAMERA" default="false" />
+    <xacro:arg name="USE_STEREO_CAMERA" default="false" />
+    <xacro:arg name="USE_AI_CAMERA" default="false" />
     <xacro:include filename="const.xacro" />
     <xacro:include filename="leg.xacro" />
@@ -14,4 +17,53 @@
         </visual>
     </link>
+    <!-- RealSense internal frames -->
+    <joint name="D435_to_camera" type="fixed">
+        <parent link="D435_camera_link" />
+        <child link="camera_link" />
+        <origin xyz="0 0 0" rpy="0 0 0" />
+    </joint>
+    <link name="camera_link" />
+    <joint name="camera_to_infra1" type="fixed">
+        <parent link="camera_link" />
+        <child link="camera_infra1_frame" />
+        <origin xyz="0 0.025 0" rpy="0 0 0" />
+    </joint>
+    <link name="camera_infra1_frame" />
+    <joint name="camera_infra1_to_optical" type="fixed">
+        <parent link="camera_infra1_frame" />
+        <child link="camera_infra1_optical_frame" />
+        <origin xyz="0 0 0" rpy="-1.5707963267948966 0 -1.5707963267948966" />
+    </joint>
+    <link name="camera_infra1_optical_frame" />
+    <joint name="camera_to_infra2" type="fixed">
+        <parent link="camera_link" />
+        <child link="camera_infra2_frame" />
+        <origin xyz="0 -0.025 0" rpy="0 0 0" />
+    </joint>
+    <link name="camera_infra2_frame" />
+    <joint name="camera_infra2_to_optical" type="fixed">
+        <parent link="camera_infra2_frame" />
+        <child link="camera_infra2_optical_frame" />
+        <origin xyz="0 0 0" rpy="-1.5707963267948966 0 -1.5707963267948966" />
+    </joint>
+    <link name="camera_infra2_optical_frame" />
+    <joint name="camera_to_depth" type="fixed">
+        <parent link="camera_link" />
+        <child link="camera_depth_frame" />
+        <origin xyz="0 0 0" rpy="0 0 0" />
+    </joint>
+    <link name="camera_depth_frame" />
+    <joint name="camera_depth_to_optical" type="fixed">
+        <parent link="camera_depth_frame" />
+        <child link="camera_depth_optical_frame" />
+        <origin xyz="0 0 0" rpy="-1.5707963267948966 0 -1.5707963267948966" />
+    </joint>
+    <link name="camera_depth_optical_frame" />
+    <joint name="camera_to_imu" type="fixed">
+        <parent link="camera_link" />
+        <child link="camera_imu_frame" />
+        <origin xyz="0 0 0" rpy="0 0 0" />
+    </joint>
+    <link name="camera_imu_frame" />
     <joint name="floating_base" type="fixed">
         <origin rpy="0 0 0" xyz="0 0 0" />
@@ -38,4 +90,10 @@
         </inertial>
     </link>
+    <joint name="RGB_camera_to_optical" type="fixed">
+        <parent link="RGB_camera_link" />
+        <child link="rgb_camera_optical_frame" />
+        <origin xyz="0 0 0" rpy="-1.5707963267948966 0 -1.5707963267948966" />
+    </joint>
+    <link name="rgb_camera_optical_frame" />
     <joint name="imu_joint" type="fixed">
         <parent link="body" />
@@ -62,4 +120,34 @@
         </collision>
     </link>
+    <joint name="AI_camera_to_optical" type="fixed">
+        <parent link="AI_camera_link" />
+        <child link="ai_camera_optical_frame" />
+        <origin xyz="0 0 0" rpy="-1.5707963267948966 0 -1.5707963267948966" />
+    </joint>
+    <link name="ai_camera_optical_frame" />
+    <joint name="body_to_left_fisheye" type="fixed">
+        <parent link="body" />
+        <child link="left_fisheye_camera_link" />
+        <origin xyz="0.095 0.125 0.100" rpy="0 0 1.5707963267948966" />
+    </joint>
+    <link name="left_fisheye_camera_link" />
+    <joint name="left_fisheye_to_optical" type="fixed">
+        <parent link="left_fisheye_camera_link" />
+        <child link="left_fisheye_camera_optical_frame" />
+        <origin xyz="0 0 0" rpy="-1.5707963267948966 0 -1.5707963267948966" />
+    </joint>
+    <link name="left_fisheye_camera_optical_frame" />
+    <joint name="body_to_right_fisheye" type="fixed">
+        <parent link="body" />
+        <child link="right_fisheye_camera_link" />
+        <origin xyz="0.095 -0.125 0.100" rpy="0 0 -1.5707963267948966" />
+    </joint>
+    <link name="right_fisheye_camera_link" />
+    <joint name="right_fisheye_to_optical" type="fixed">
+        <parent link="right_fisheye_camera_link" />
+        <child link="right_fisheye_camera_optical_frame" />
+        <origin xyz="0 0 0" rpy="-1.5707963267948966 0 -1.5707963267948966" />
+    </joint>
+    <link name="right_fisheye_camera_optical_frame" />
     <joint name="scan_joint" type="fixed">
         <parent link="body" />
